File: shield/schematic.sch (EAGLE design)
At the start: 63 parts, among them IC1 LM358N, IC2 LM358N

Commit message: Update
Other:
- note added: "Designed by LONGUET Gilles June 2014"
- note removed: "Designed by LONGUET Gilles June 2013"
Changed lines of the file:
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@@
 <grid distance="0.1" unitdist="inch" unit="inch" style="lines" multiple="1" display="no" altdistance="0.01" altunitdist="inch" altunit="inch"/>
 <layers>
-<layer number="1" name="Top" color="4" fill="1" visible="yes" active="no"/>
-<layer number="2" name="Route2" color="1" fill="3" visible="yes" active="no"/>
-<layer number="3" name="Route3" color="4" fill="3" visible="yes" active="no"/>
-<layer number="4" name="Route4" color="1" fill="4" visible="yes" active="no"/>
-<layer number="5" name="Route5" color="4" fill="4" visible="yes" active="no"/>
-<layer number="6" name="Route6" color="1" fill="8" visible="yes" active="no"/>
-<layer number="7" name="Route7" color="4" fill="8" visible="yes" active="no"/>
-<layer number="8" name="Route8" color="1" fill="2" visible="yes" active="no"/>
-<layer number="9" name="Route9" color="4" fill="2" visible="yes" active="no"/>
-<layer number="10" name="Route10" color="1" fill="7" visible="yes" active="no"/>
-<layer number="11" name="Route11" color="4" fill="7" visible="yes" active="no"/>
-<layer number="12" name="Route12" color="1" fill="5" visible="yes" active="no"/>
-<layer number="13" name="Route13" color="4" fill="5" visible="yes" active="no"/>
-<layer number="14" name="Route14" color="1" fill="6" visible="yes" active="no"/>
-<layer number="15" name="Route15" color="4" fill="6" visible="yes" active="no"/>
-<layer number="16" name="Bottom" color="1" fill="1" visible="yes" active="no"/>
-<layer number="17" name="Pads" color="2" fill="1" visible="yes" active="no"/>
-<layer number="18" name="Vias" color="14" fill="1" visible="yes" active="no"/>
-<layer number="19" name="Unrouted" color="6" fill="1" visible="yes" active="no"/>
-<layer number="20" name="Dimension" color="15" fill="1" visible="yes" active="no"/>
-<layer number="21" name="tPlace" color="7" fill="1" visible="yes" active="no"/>
-<layer number="22" name="bPlace" color="7" fill="1" visible="yes" active="no"/>
-<layer number="23" name="tOrigins" color="15" fill="1" visible="yes" active="no"/>
-<layer number="24" name="bOrigins" color="15" fill="1" visible="yes" active="no"/>
-<layer number="25" name="tNames" color="7" fill="1" visible="yes" active="no"/>
-<layer number="26" name="bNames" color="7" fill="1" visible="yes" active="no"/>
-<layer number="27" name="tValues" color="7" fill="1" visible="yes" active="no"/>
-<layer number="28" name="bValues" color="7" fill="1" visible="yes" active="no"/>
+<layer number="1" name="Top" color="4" fill="1" visible="no" active="no"/>
+<layer number="2" name="Route2" color="1" fill="3" visible="no" active="no"/>
+<layer number="3" name="Route3" color="4" fill="3" visible="no" active="no"/>
+<layer number="4" name="Route4" color="1" fill="4" visible="no" active="no"/>
+<layer number="5" name="Route5" color="4" fill="4" visible="no" active="no"/>
+<layer number="6" name="Route6" color="1" fill="8" visible="no" active="no"/>
+<layer number="7" name="Route7" color="4" fill="8" visible="no" active="no"/>
+<layer number="8" name="Route8" color="1" fill="2" visible="no" active="no"/>
+<layer number="9" name="Route9" color="4" fill="2" visible="no" active="no"/>
+<layer number="10" name="Route10" color="1" fill="7" visible="no" active="no"/>
+<layer number="11" name="Route11" color="4" fill="7" visible="no" active="no"/>
+<layer number="12" name="Route12" color="1" fill="5" visible="no" active="no"/>
+<layer number="13" name="Route13" color="4" fill="5" visible="no" active="no"/>
+<layer number="14" name="Route14" color="1" fill="6" visible="no" active="no"/>
+<layer number="15" name="Route15" color="4" fill="6" visible="no" active="no"/>
+<layer number="16" name="Bottom" color="1" fill="1" visible="no" active="no"/>
+<layer number="17" name="Pads" color="2" fill="1" visible="no" active="no"/>
+<layer number="18" name="Vias" color="14" fill="1" visible="no" active="no"/>
+<layer number="19" name="Unrouted" color="6" fill="1" visible="no" active="no"/>
+<layer number="20" name="Dimension" color="15" fill="1" visible="no" active="no"/>
+<layer number="21" name="tPlace" color="7" fill="1" visible="no" active="no"/>
+<layer number="22" name="bPlace" color="7" fill="1" visible="no" active="no"/>
+<layer number="23" name="tOrigins" color="15" fill="1" visible="no" active="no"/>
+<layer number="24" name="bOrigins" color="15" fill="1" visible="no" active="no"/>
+<layer number="25" name="tNames" color="7" fill="1" visible="no" active="no"/>
+<layer number="26" name="bNames" color="7" fill="1" visible="no" active="no"/>
+<layer number="27" name="tValues" color="7" fill="1" visible="no" active="no"/>
+<layer number="28" name="bValues" color="7" fill="1" visible="no" active="no"/>
 <layer number="29" name="tStop" color="2" fill="3" visible="no" active="no"/>
 <layer number="30" name="bStop" color="5" fill="6" visible="no" active="no"/>
@@
 <layer number="35" name="tGlue" color="7" fill="4" visible="no" active="no"/>
 <layer number="36" name="bGlue" color="7" fill="5" visible="no" active="no"/>
-<layer number="37" name="tTest" color="7" fill="1" visible="yes" active="no"/>
-<layer number="38" name="bTest" color="7" fill="1" visible="yes" active="no"/>
+<layer number="37" name="tTest" color="7" fill="1" visible="no" active="no"/>
+<layer number="38" name="bTest" color="7" fill="1" visible="no" active="no"/>
 <layer number="39" name="tKeepout" color="4" fill="11" visible="no" active="no"/>
 <layer number="40" name="bKeepout" color="1" fill="11" visible="no" active="no"/>
@@
 <layer number="44" name="Drills" color="7" fill="1" visible="no" active="no"/>
 <layer number="45" name="Holes" color="7" fill="1" visible="no" active="no"/>
-<layer number="46" name="Milling" color="3" fill="1" visible="yes" active="no"/>
-<layer number="47" name="Measures" color="7" fill="1" visible="yes" active="no"/>
-<layer number="48" name="Document" color="7" fill="1" visible="yes" active="no"/>
-<layer number="49" name="Reference" color="13" fill="1" visible="yes" active="no"/>
-<layer number="50" name="dxf" color="12" fill="1" visible="yes" active="no"/>
-<layer number="51" name="tDocu" color="7" fill="1" visible="yes" active="no"/>
-<layer number="52" name="bDocu" color="7" fill="1" visible="yes" active="no"/>
-<layer number="53" name="tGND_GNDA" color="7" fill="9" visible="yes" active="no"/>
-<layer number="54" name="bGND_GNDA" color="1" fill="9" visible="yes" active="no"/>
-<layer number="56" name="wert" color="7" fill="1" visible="yes" active="no"/>
-<layer number="57" name="tCAD" color="7" fill="1" visible="yes" active="no"/>
+<layer number="46" name="Milling" color="3" fill="1" visible="no" active="no"/>
+<layer number="47" name="Measures" color="7" fill="1" visible="no" active="no"/>
+<layer number="48" name="Document" color="7" fill="1" visible="no" active="no"/>
+<layer number="49" name="Reference" color="13" fill="1" visible="no" active="no"/>
+<layer number="50" name="dxf" color="12" fill="1" visible="no" active="no"/>
+<layer number="51" name="tDocu" color="7" fill="1" visible="no" active="no"/>
+<layer number="52" name="bDocu" color="7" fill="1" visible="no" active="no"/>
+<layer number="53" name="tGND_GNDA" color="7" fill="9" visible="no" active="no"/>
+<layer number="54" name="bGND_GNDA" color="1" fill="9" visible="no" active="no"/>
+<layer number="56" name="wert" color="7" fill="1" visible="no" active="no"/>
+<layer number="57" name="tCAD" color="7" fill="1" visible="no" active="no"/>
 <layer number="91" name="Nets" color="2" fill="1" visible="yes" active="yes"/>
 <layer number="92" name="Busses" color="1" fill="1" visible="yes" active="yes"/>
@@
 <text x="146.05" y="265.43" size="1.778" layer="91">since Arduino Etherent shield also uses Dig10</text>
 <text x="-30.48" y="213.36" size="1.778" layer="91">NetBomo : github.com/netbomo/alpha1</text>
-<text x="-30.48" y="208.28" size="1.778" layer="91">Designed by LONGUET Gilles June 2013</text>
+<text x="-30.48" y="208.28" size="1.778" layer="91">Designed by LONGUET Gilles June 2014</text>
 <text x="17.78" y="208.28" size="1.778" layer="91">Based on openenergymonitor.org</text>
 </plain>

Commit message: update shematic.sch
Parts:
- removed ANEMO: 1X4-3.5MM, adafruit:1X4-3.5MM
- added ANEMO1, ANEMO2: 1X4-3.5MM, adafruit:1X4-3.5MM
- added R22, R23: 10k, rcl:R-EU_0204/7
Connections:
- net +5V: now also R22.2, R23.2
- net ANEMO1A: now also ANEMO1.1; no longer ANEMO.1
- net ANEMO1B: now also ANEMO1.2; no longer ANEMO.2
- net ANEMO2: now also ANEMO2.3, R23.1
- net ANEMO2A: now also ANEMO2.1; no longer ANEMO.3
- net ANEMO2B: now also ANEMO2.2; no longer ANEMO.4
- net DIG3: now also ANEMO1.3, R22.1
- net GND: now also ANEMO1.4, ANEMO2.4
Other:
- moved on the sheet: R17, R21, WINDVANE
Changed lines of the file:
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@@
 <part name="U$4" library="JeeParts" deviceset="RFM12B" device=""/>
 <part name="U$2" library="adafruit" deviceset="ARDUINO" device="-BPLACE"/>
-<part name="ANEMO" library="adafruit" deviceset="1X4" device="-3.5MM"/>
 <part name="WINDVANE" library="adafruit" deviceset="1X4" device="-3.5MM"/>
 <part name="R17" library="rcl" deviceset="R-EU_" device="0204/7" value="10k"/>
 <part name="R21" library="rcl" deviceset="R-EU_" device="0204/7" value="10k"/>
 <part name="P+5" library="supply1" deviceset="+5V" device=""/>
+<part name="ANEMO1" library="adafruit" deviceset="1X4" device="-3.5MM"/>
+<part name="ANEMO2" library="adafruit" deviceset="1X4" device="-3.5MM"/>
+<part name="R22" library="rcl" deviceset="R-EU_" device="0204/7" value="10k"/>
+<part name="R23" library="rcl" deviceset="R-EU_" device="0204/7" value="10k"/>
+<part name="P+11" library="supply1" deviceset="+5V" device=""/>
+<part name="P+14" library="supply1" deviceset="+5V" device=""/>
 </parts>
 <sheets>
@@
 <instance part="U$4" gate="G$1" x="147.32" y="217.17"/>
 <instance part="U$2" gate="G$1" x="144.78" y="321.31" rot="R270"/>
-<instance part="ANEMO" gate="G$1" x="-66.04" y="373.38" rot="MR0"/>
-<instance part="WINDVANE" gate="G$1" x="-66.04" y="347.98" rot="MR0"/>
-<instance part="R17" gate="G$1" x="-58.42" y="355.6" rot="R90"/>
-<instance part="R21" gate="G$1" x="-48.26" y="340.36" rot="R90"/>
-<instance part="P+5" gate="1" x="-58.42" y="365.76"/>
+<instance part="WINDVANE" gate="G$1" x="-63.5" y="294.64" rot="MR0"/>
+<instance part="R17" gate="G$1" x="-55.88" y="302.26" rot="R90"/>
+<instance part="R21" gate="G$1" x="-45.72" y="287.02" rot="R90"/>
+<instance part="P+5" gate="1" x="-55.88" y="312.42"/>
+<instance part="ANEMO1" gate="G$1" x="-63.5" y="373.38" rot="MR0"/>
+<instance part="ANEMO2" gate="G$1" x="-63.5" y="347.98" rot="MR0"/>
+<instance part="R22" gate="G$1" x="76.2" y="363.22" rot="R90"/>
+<instance part="R23" gate="G$1" x="66.04" y="325.12" rot="R90"/>
+<instance part="P+11" gate="1" x="76.2" y="373.38"/>
+<instance part="P+14" gate="1" x="66.04" y="335.28"/>
 </instances>
 <busses>
@@
 <pinref part="P+5" gate="1" pin="+5V"/>
 <pinref part="R17" gate="G$1" pin="2"/>
-<wire x1="-58.42" y1="363.22" x2="-58.42" y2="360.68" width="0.1524" layer="91"/>
+<wire x1="-55.88" y1="309.88" x2="-55.88" y2="307.34" width="0.1524" layer="91"/>
+</segment>
+<segment>
+<pinref part="P+11" gate="1" pin="+5V"/>
+<pinref part="R22" gate="G$1" pin="2"/>
+<wire x1="76.2" y1="370.84" x2="76.2" y2="368.3" width="0.1524" layer="91"/>
+</segment>
+<segment>
+<pinref part="P+14" gate="1" pin="+5V"/>
+<pinref part="R23" gate="G$1" pin="2"/>
+<wire x1="66.04" y1="332.74" x2="66.04" y2="330.2" width="0.1524" layer="91"/>
 </segment>
 </net>
@@
 <segment>
 <pinref part="WINDVANE" gate="G$1" pin="4"/>
-<wire x1="-60.96" y1="342.9" x2="-58.42" y2="342.9" width="0.1524" layer="91"/>
-<label x="-55.88" y="342.9" size="1.778" layer="95"/>
+<wire x1="-58.42" y1="289.56" x2="-55.88" y2="289.56" width="0.1524" layer="91"/>
+<label x="-53.34" y="289.56" size="1.778" layer="95"/>
 <pinref part="R21" gate="G$1" pin="1"/>
-<wire x1="-58.42" y1="342.9" x2="-53.34" y2="342.9" width="0.1524" layer="91"/>
-<wire x1="-48.26" y1="335.28" x2="-58.42" y2="335.28" width="0.1524" layer="91"/>
-<wire x1="-58.42" y1="335.28" x2="-58.42" y2="342.9" width="0.1524" layer="91"/>
-<junction x="-58.42" y="342.9"/>
+<wire x1="-55.88" y1="289.56" x2="-50.8" y2="289.56" width="0.1524" layer="91"/>
+<wire x1="-45.72" y1="281.94" x2="-55.88" y2="281.94" width="0.1524" layer="91"/>
+<wire x1="-55.88" y1="281.94" x2="-55.88" y2="289.56" width="0.1524" layer="91"/>
+<junction x="-55.88" y="289.56"/>
+</segment>
+<segment>
+<pinref part="ANEMO1" gate="G$1" pin="4"/>
+<wire x1="-48.26" y1="368.3" x2="-58.42" y2="368.3" width="0.1524" layer="91"/>
+<label x="-48.26" y="368.3" size="1.778" layer="95"/>
+</segment>
+<segment>
+<pinref part="ANEMO2" gate="G$1" pin="4"/>
+<wire x1="-48.26" y1="342.9" x2="-58.42" y2="342.9" width="0.1524" layer="91"/>
+<label x="-48.26" y="342.9" size="1.778" layer="95"/>
 </segment>
 </net>
@@
 <segment>
 <pinref part="WINDVANE" gate="G$1" pin="2"/>
-<wire x1="-60.96" y1="347.98" x2="-53.34" y2="347.98" width="0.1524" layer="91"/>
-<label x="-55.88" y="347.98" size="1.778" layer="95"/>
+<wire x1="-58.42" y1="294.64" x2="-50.8" y2="294.64" width="0.1524" layer="91"/>
+<label x="-53.34" y="294.64" size="1.778" layer="95"/>
 </segment>
 </net>
@@
 <wire x1="68.58" y1="355.6" x2="68.58" y2="345.44" width="0.1524" layer="91"/>
 <wire x1="68.58" y1="345.44" x2="63.5" y2="345.44" width="0.1524" layer="91"/>
-<wire x1="68.58" y1="355.6" x2="73.66" y2="355.6" width="0.1524" layer="91"/>
-<label x="73.66" y="355.6" size="1.778" layer="95"/>
+<wire x1="68.58" y1="355.6" x2="76.2" y2="355.6" width="0.1524" layer="91"/>
+<label x="86.36" y="355.6" size="1.778" layer="95"/>
 <junction x="68.58" y="355.6"/>
+<pinref part="R22" gate="G$1" pin="1"/>
+<wire x1="76.2" y1="355.6" x2="88.9" y2="355.6" width="0.1524" layer="91"/>
+<wire x1="76.2" y1="358.14" x2="76.2" y2="355.6" width="0.1524" layer="91"/>
+<junction x="76.2" y="355.6"/>
+</segment>
+<segment>
+<pinref part="ANEMO1" gate="G$1" pin="3"/>
+<wire x1="-48.26" y1="370.84" x2="-58.42" y2="370.84" width="0.1524" layer="91"/>
+<label x="-48.26" y="370.84" size="1.778" layer="95"/>
 </segment>
 </net>
@@
 <pinref part="IC1" gate="B" pin="OUT"/>
 <wire x1="58.42" y1="317.5" x2="60.96" y2="317.5" width="0.1524" layer="91"/>
-<wire x1="60.96" y1="317.5" x2="71.12" y2="317.5" width="0.1524" layer="91"/>
+<wire x1="60.96" y1="317.5" x2="66.04" y2="317.5" width="0.1524" layer="91"/>
+<wire x1="66.04" y1="317.5" x2="76.2" y2="317.5" width="0.1524" layer="91"/>
 <wire x1="60.96" y1="307.34" x2="60.96" y2="317.5" width="0.1524" layer="91"/>
 <junction x="60.96" y="317.5"/>
-<label x="66.04" y="317.5" size="1.778" layer="95"/>
+<label x="71.12" y="317.5" size="1.778" layer="95"/>
+<pinref part="R23" gate="G$1" pin="1"/>
+<wire x1="66.04" y1="320.04" x2="66.04" y2="317.5" width="0.1524" layer="91"/>
+<junction x="66.04" y="317.5"/>
 </segment>
 <segment>
@@
 <wire x1="137.16" y1="177.8" x2="121.92" y2="177.8" width="0.1524" layer="91"/>
 <label x="121.92" y="177.8" size="1.778" layer="95"/>
+</segment>
+<segment>
+<pinref part="ANEMO2" gate="G$1" pin="3"/>
+<wire x1="-48.26" y1="345.44" x2="-58.42" y2="345.44" width="0.1524" layer="91"/>
+<label x="-48.26" y="345.44" size="1.778" layer="95"/>
 </segment>
 </net>
@@
 <net name="ANEMO1A" class="0">
 <segment>
-<pinref part="ANEMO" gate="G$1" pin="1"/>
-<wire x1="-60.96" y1="375.92" x2="-53.34" y2="375.92" width="0.1524" layer="91"/>
-<label x="-55.88" y="375.92" size="1.778" layer="95"/>
-</segment>
-<segment>
 <pinref part="R31" gate="G$1" pin="1"/>
 <wire x1="-25.4" y1="360.68" x2="-35.56" y2="360.68" width="0.1524" layer="91"/>
 <label x="-43.18" y="360.68" size="1.778" layer="95"/>
 </segment>
+<segment>
+<pinref part="ANEMO1" gate="G$1" pin="1"/>
+<wire x1="-58.42" y1="375.92" x2="-48.26" y2="375.92" width="0.1524" layer="91"/>
+<label x="-48.26" y="375.92" size="1.778" layer="95"/>
+</segment>
 </net>
 <net name="ANEMO1B" class="0">
-<segment>
-<pinref part="ANEMO" gate="G$1" pin="2"/>
-<wire x1="-60.96" y1="373.38" x2="-53.34" y2="373.38" width="0.1524" layer="91"/>
-<label x="-55.88" y="373.38" size="1.778" layer="95"/>
-</segment>
 <segment>
 <pinref part="R32" gate="G$1" pin="1"/>
@@
 <label x="-43.18" y="355.6" size="1.778" layer="95"/>
 </segment>
+<segment>
+<pinref part="ANEMO1" gate="G$1" pin="2"/>
+<wire x1="-48.26" y1="373.38" x2="-58.42" y2="373.38" width="0.1524" layer="91"/>
+<label x="-48.26" y="373.38" size="1.778" layer="95"/>
+</segment>
 </net>
 <net name="ANEMO2A" class="0">
-<segment>
-<pinref part="ANEMO" gate="G$1" pin="3"/>
-<wire x1="-60.96" y1="370.84" x2="-53.34" y2="370.84" width="0.1524" layer="91"/>
-<label x="-55.88" y="370.84" size="1.778" layer="95"/>
-</segment>
 <segment>
 <pinref part="R40" gate="G$1" pin="1"/>
@@
 <label x="-48.26" y="322.58" size="1.778" layer="95"/>
 </segment>
+<segment>
+<pinref part="ANEMO2" gate="G$1" pin="1"/>
+<wire x1="-48.26" y1="350.52" x2="-58.42" y2="350.52" width="0.1524" layer="91"/>
+<label x="-48.26" y="350.52" size="1.778" layer="95"/>
+</segment>
 </net>
 <net name="ANEMO2B" class="0">
-<segment>
-<pinref part="ANEMO" gate="G$1" pin="4"/>
-<wire x1="-60.96" y1="368.3" x2="-53.34" y2="368.3" width="0.1524" layer="91"/>
-<label x="-55.88" y="368.3" size="1.778" layer="95"/>
-</segment>
 <segment>
 <pinref part="R41" gate="G$1" pin="1"/>
@@
 <label x="-48.26" y="317.5" size="1.778" layer="95"/>
 </segment>
+<segment>
+<pinref part="ANEMO2" gate="G$1" pin="2"/>
+<wire x1="-48.26" y1="347.98" x2="-58.42" y2="347.98" width="0.1524" layer="91"/>
+<label x="-48.26" y="347.98" size="1.778" layer="95"/>
+</segment>
 </net>
 <net name="N$3" class="0">
@@
 <pinref part="R17" gate="G$1" pin="1"/>
 <pinref part="WINDVANE" gate="G$1" pin="1"/>
-<wire x1="-58.42" y1="350.52" x2="-60.96" y2="350.52" width="0.1524" layer="91"/>
+<wire x1="-55.88" y1="297.18" x2="-58.42" y2="297.18" width="0.1524" layer="91"/>
 </segment>
 </net>
@@
 <pinref part="WINDVANE" gate="G$1" pin="3"/>
 <pinref part="R21" gate="G$1" pin="2"/>
-<wire x1="-60.96" y1="345.44" x2="-48.26" y2="345.44" width="0.1524" layer="91"/>
-</segment>
-</net>
+<wire x1="-58.42" y1="292.1" x2="-45.72" y2="292.1" width="0.1524" layer="91"/>
+</segment>
+</net>
