File: shield/kicad files/netbomo.sch (KiCad schematic (older format))
At the start: 53 parts, among them CON1 BARREL_JACK, J1 JACK_STEREO, P1 WIND1, P2 WIND2, P3 VANE, P5 WIND2/RFM, U1 LM358, U2 LM358, U3 RFM12

Commit message: update kicad files
Parts:
- renumbered CON1 to 9VAC1, J1 to CT1, U3 to RFM12
Connections:
- wire segments 179 -> 184
Changed lines of the file:
@@
 P 9100 2350
 F 0 "SHIELD1" H 8750 3300 60  0000 C CNN
-F 1 "ARDUINO_SHIELD" H 9150 1400 60  0000 C CNN
+F 1 "ARDUINO_SHIELD" H 9400 3300 60  0000 C CNN
 F 2 "Arduino:ARDUINO_SHIELD_2" H 9100 2350 60  0001 C CNN
 F 3 "" H 9100 2350 60  0000 C CNN
@@
 $EndComp
 $Comp
-L RFM12 U3
-U 1 1 546EF88E
+L RFM12 RFM12
+U 2 1 546EF88E
 P 8650 5550
-F 0 "U3" V 8650 5550 60  0000 C CNN
+F 0 "RFM12" H 8650 5550 60  0000 C CNN
 F 1 "RFM12" H 9044 5944 60  0000 C CNN
 F 2 "rfm12:RFM12" H 8650 5550 60  0001 C CNN
 F 3 "" H 8650 5550 60  0000 C CNN
-	1    8650 5550
-	1    0    0    -1
-$EndComp
-$Comp
-L VPP #PWR28
+	2    8650 5550
+	1    0    0    -1
+$EndComp
+$Comp
+L VPP #PWR31
 U 1 1 546EF961
 P 9950 5750
-F 0 "#PWR28" H 9950 5950 40  0001 C CNN
+F 0 "#PWR31" H 9950 5950 40  0001 C CNN
 F 1 "ANT" H 9950 5900 40  0000 C CNN
 F 2 "" H 9950 5750 60  0000 C CNN
@@
 $EndComp
 $Comp
-L +3.3V #PWR01
+L +3.3V #PWR34
 U 1 1 546EFAB4
 P 10950 4400
-F 0 "#PWR01" H 10950 4360 30  0001 C CNN
+F 0 "#PWR34" H 10950 4360 30  0001 C CNN
 F 1 "+3.3V" H 10950 4510 30  0000 C CNN
 F 2 "" H 10950 4400 60  0000 C CNN
@@
 $EndComp
 $Comp
-L +3.3V #PWR02
+L +3.3V #PWR28
 U 1 1 546EFACA
 P 8650 4950
-F 0 "#PWR02" H 8650 4910 30  0001 C CNN
+F 0 "#PWR28" H 8650 4910 30  0001 C CNN
 F 1 "+3.3V" H 8650 5060 30  0000 C CNN
 F 2 "" H 8650 4950 60  0000 C CNN
@@
 $EndComp
 $Comp
-L GND #PWR03
+L GND #PWR35
 U 1 1 546EFAE0
 P 10950 5550
-F 0 "#PWR03" H 10950 5550 30  0001 C CNN
+F 0 "#PWR35" H 10950 5550 30  0001 C CNN
 F 1 "GND" H 10950 5480 30  0001 C CNN
 F 2 "" H 10950 5550 60  0000 C CNN
@@
 $EndComp
 $Comp
-L GND #PWR04
+L GND #PWR29
 U 1 1 546EFAF6
 P 8750 6200
-F 0 "#PWR04" H 8750 6200 30  0001 C CNN
+F 0 "#PWR29" H 8750 6200 30  0001 C CNN
 F 1 "GND" H 8750 6130 30  0001 C CNN
 F 2 "" H 8750 6200 60  0000 C CNN
@@
 $EndComp
 $Comp
-L GND #PWR05
+L GND #PWR3
 U 1 1 546F0EDA
 P 1500 1050
-F 0 "#PWR05" H 1500 1050 30  0001 C CNN
+F 0 "#PWR3" H 1500 1050 30  0001 C CNN
 F 1 "GND" H 1500 980 30  0001 C CNN
 F 2 "" H 1500 1050 60  0000 C CNN
@@
 $EndComp
 $Comp
-L GND #PWR06
+L GND #PWR6
 U 1 1 546F0F09
 P 2250 1950
-F 0 "#PWR06" H 2250 1950 30  0001 C CNN
+F 0 "#PWR6" H 2250 1950 30  0001 C CNN
 F 1 "GND" H 2250 1880 30  0001 C CNN
 F 2 "" H 2250 1950 60  0000 C CNN
@@
 $EndComp
 $Comp
-L GND #PWR07
+L GND #PWR18
 U 1 1 546F0F38
 P 4850 2050
-F 0 "#PWR07" H 4850 2050 30  0001 C CNN
+F 0 "#PWR18" H 4850 2050 30  0001 C CNN
 F 1 "GND" H 4850 1980 30  0001 C CNN
 F 2 "" H 4850 2050 60  0000 C CNN
@@
 $EndComp
 $Comp
-L +5V #PWR08
+L +5V #PWR5
 U 1 1 546F0FB8
 P 2250 1050
-F 0 "#PWR08" H 2250 1140 20  0001 C CNN
+F 0 "#PWR5" H 2250 1140 20  0001 C CNN
 F 1 "+5V" H 2250 1140 30  0000 C CNN
 F 2 "" H 2250 1050 60  0000 C CNN
@@
 $EndComp
 $Comp
-L +5V #PWR09
+L +5V #PWR17
 U 1 1 546F0FE7
 P 4850 1150
-F 0 "#PWR09" H 4850 1240 20  0001 C CNN
+F 0 "#PWR17" H 4850 1240 20  0001 C CNN
 F 1 "+5V" H 4850 1240 30  0000 C CNN
 F 2 "" H 4850 1150 60  0000 C CNN
@@
 $EndComp
 $Comp
-L +5V #PWR010
+L +5V #PWR15
 U 1 1 546F1016
 P 4300 900
-F 0 "#PWR010" H 4300 990 20  0001 C CNN
+F 0 "#PWR15" H 4300 990 20  0001 C CNN
 F 1 "+5V" H 4300 990 30  0000 C CNN
 F 2 "" H 4300 900 60  0000 C CNN
@@
 $EndComp
 $Comp
-L +5V #PWR011
+L +5V #PWR23
 U 1 1 546F1096
 P 5650 950
-F 0 "#PWR011" H 5650 1040 20  0001 C CNN
+F 0 "#PWR23" H 5650 1040 20  0001 C CNN
 F 1 "+5V" H 5650 1040 30  0000 C CNN
 F 2 "" H 5650 950 60  0000 C CNN
@@
 $EndComp
 $Comp
-L GND #PWR012
+L GND #PWR1
 U 1 1 546F5877
 P 950 1850
-F 0 "#PWR012" H 950 1850 30  0001 C CNN
+F 0 "#PWR1" H 950 1850 30  0001 C CNN
 F 1 "GND" H 950 1780 30  0001 C CNN
 F 2 "" H 950 1850 60  0000 C CNN
@@
 $EndComp
 $Comp
-L GND #PWR013
+L GND #PWR32
 U 1 1 54777EB5
 P 10350 6350
-F 0 "#PWR013" H 10350 6350 30  0001 C CNN
+F 0 "#PWR32" H 10350 6350 30  0001 C CNN
 F 1 "GND" H 10350 6280 30  0001 C CNN
 F 2 "" H 10350 6350 60  0000 C CNN
@@
 $EndComp
 $Comp
-L GND #PWR014
+L GND #PWR36
 U 1 1 5477CF77
 P 11000 3300
-F 0 "#PWR014" H 11000 3300 30  0001 C CNN
+F 0 "#PWR36" H 11000 3300 30  0001 C CNN
 F 1 "GND" H 11000 3230 30  0001 C CNN
 F 2 "" H 11000 3300 60  0000 C CNN
@@
 $EndComp
 $Comp
-L GND #PWR015
+L GND #PWR14
 U 1 1 5477D805
 P 3800 7500
-F 0 "#PWR015" H 3800 7500 30  0001 C CNN
+F 0 "#PWR14" H 3800 7500 30  0001 C CNN
 F 1 "GND" H 3800 7430 30  0001 C CNN
 F 2 "" H 3800 7500 60  0000 C CNN
@@
 $EndComp
 $Comp
-L +5V #PWR016
+L +5V #PWR11
 U 1 1 5477D846
 P 3150 6700
-F 0 "#PWR016" H 3150 6790 20  0001 C CNN
+F 0 "#PWR11" H 3150 6790 20  0001 C CNN
 F 1 "+5V" H 3150 6790 30  0000 C CNN
 F 2 "" H 3150 6700 60  0000 C CNN
@@
 $EndComp
 $Comp
-L GND #PWR017
+L GND #PWR10
 U 1 1 54781C1E
 P 2750 5850
-F 0 "#PWR017" H 2750 5850 30  0001 C CNN
+F 0 "#PWR10" H 2750 5850 30  0001 C CNN
 F 1 "GND" H 2750 5780 30  0001 C CNN
 F 2 "" H 2750 5850 60  0000 C CNN
@@
 $EndComp
 $Comp
-L +5V #PWR018
+L +5V #PWR9
 U 1 1 54781C66
 P 2750 4550
-F 0 "#PWR018" H 2750 4640 20  0001 C CNN
+F 0 "#PWR9" H 2750 4640 20  0001 C CNN
 F 1 "+5V" H 2750 4640 30  0000 C CNN
 F 2 "" H 2750 4550 60  0000 C CNN
@@
 $EndComp
 $Comp
-L GND #PWR019
+L GND #PWR4
 U 1 1 54787CEB
 P 1500 2650
-F 0 "#PWR019" H 1500 2650 30  0001 C CNN
+F 0 "#PWR4" H 1500 2650 30  0001 C CNN
 F 1 "GND" H 1500 2580 30  0001 C CNN
 F 2 "" H 1500 2650 60  0000 C CNN
@@
 $EndComp
 $Comp
-L GND #PWR020
+L GND #PWR8
 U 1 1 54787CF1
 P 2250 3550
-F 0 "#PWR020" H 2250 3550 30  0001 C CNN
+F 0 "#PWR8" H 2250 3550 30  0001 C CNN
 F 1 "GND" H 2250 3480 30  0001 C CNN
 F 2 "" H 2250 3550 60  0000 C CNN
@@
 $EndComp
 $Comp
-L GND #PWR021
+L GND #PWR20
 U 1 1 54787CF7
 P 4850 3650
-F 0 "#PWR021" H 4850 3650 30  0001 C CNN
+F 0 "#PWR20" H 4850 3650 30  0001 C CNN
 F 1 "GND" H 4850 3580 30  0001 C CNN
 F 2 "" H 4850 3650 60  0000 C CNN
@@
 $EndComp
 $Comp
-L +5V #PWR022
+L +5V #PWR7
 U 1 1 54787CFD
 P 2250 2650
-F 0 "#PWR022" H 2250 2740 20  0001 C CNN
+F 0 "#PWR7" H 2250 2740 20  0001 C CNN
 F 1 "+5V" H 2250 2740 30  0000 C CNN
 F 2 "" H 2250 2650 60  0000 C CNN
@@
 $EndComp
 $Comp
-L +5V #PWR023
+L +5V #PWR19
 U 1 1 54787D03
 P 4850 2750
-F 0 "#PWR023" H 4850 2840 20  0001 C CNN
+F 0 "#PWR19" H 4850 2840 20  0001 C CNN
 F 1 "+5V" H 4850 2840 30  0000 C CNN
 F 2 "" H 4850 2750 60  0000 C CNN
@@
 $EndComp
 $Comp
-L +5V #PWR024
+L +5V #PWR16
 U 1 1 54787D09
 P 4300 2500
-F 0 "#PWR024" H 4300 2590 20  0001 C CNN
+F 0 "#PWR16" H 4300 2590 20  0001 C CNN
 F 1 "+5V" H 4300 2590 30  0000 C CNN
 F 2 "" H 4300 2500 60  0000 C CNN
@@
 $EndComp
 $Comp
-L +5V #PWR025
+L +5V #PWR24
 U 1 1 54787D0F
 P 5650 2550
-F 0 "#PWR025" H 5650 2640 20  0001 C CNN
+F 0 "#PWR24" H 5650 2640 20  0001 C CNN
 F 1 "+5V" H 5650 2640 30  0000 C CNN
 F 2 "" H 5650 2550 60  0000 C CNN
@@
 $EndComp
 $Comp
-L GND #PWR026
+L GND #PWR2
 U 1 1 54787D1C
 P 950 3450
-F 0 "#PWR026" H 950 3450 30  0001 C CNN
+F 0 "#PWR2" H 950 3450 30  0001 C CNN
 F 1 "GND" H 950 3380 30  0001 C CNN
 F 2 "" H 950 3450 60  0000 C CNN
@@
 $EndComp
 $Comp
-L +5V #PWR027
+L +5V #PWR21
 U 1 1 54790DDF
 P 5250 4150
-F 0 "#PWR027" H 5250 4240 20  0001 C CNN
+F 0 "#PWR21" H 5250 4240 20  0001 C CNN
 F 1 "+5V" H 5250 4240 30  0000 C CNN
 F 2 "" H 5250 4150 60  0000 C CNN
@@
 $EndComp
 $Comp
-L GND #PWR028
+L GND #PWR22
 U 1 1 54791019
 P 5250 5800
-F 0 "#PWR028" H 5250 5800 30  0001 C CNN
+F 0 "#PWR22" H 5250 5800 30  0001 C CNN
 F 1 "GND" H 5250 5730 30  0001 C CNN
 F 2 "" H 5250 5800 60  0000 C CNN
@@
 ADC3
 $Comp
-L GND #PWR029
+L GND #PWR33
 U 1 1 5479E9F2
 P 10650 1750
-F 0 "#PWR029" H 10650 1750 30  0001 C CNN
+F 0 "#PWR33" H 10650 1750 30  0001 C CNN
 F 1 "GND" H 10650 1680 30  0001 C CNN
 F 2 "" H 10650 1750 60  0000 C CNN
@@
 $EndComp
 $Comp
-L GND #PWR030
+L GND #PWR27
 U 1 1 5479EA3D
 P 7550 2400
-F 0 "#PWR030" H 7550 2400 30  0001 C CNN
+F 0 "#PWR27" H 7550 2400 30  0001 C CNN
 F 1 "GND" H 7550 2330 30  0001 C CNN
 F 2 "" H 7550 2400 60  0000 C CNN
@@
 $EndComp
 $Comp
-L +5V #PWR031
+L +5V #PWR25
 U 1 1 5479EA88
 P 7400 1950
-F 0 "#PWR031" H 7400 2040 20  0001 C CNN
+F 0 "#PWR25" H 7400 2040 20  0001 C CNN
 F 1 "+5V" H 7400 2040 30  0000 C CNN
 F 2 "" H 7400 1950 60  0000 C CNN
@@
 $EndComp
 $Comp
-L +3.3V #PWR032
+L +3.3V #PWR26
 U 1 1 5479EAD3
 P 7550 1950
-F 0 "#PWR032" H 7550 1910 30  0001 C CNN
+F 0 "#PWR26" H 7550 1910 30  0001 C CNN
 F 1 "+3.3V" H 7550 2060 30  0000 C CNN
 F 2 "" H 7550 1950 60  0000 C CNN
@@
 NoConn ~ 1950 5300
 $Comp
-L BARREL_JACK CON1
+L BARREL_JACK 9VAC1
 U 1 1 547BC53E
 P 5600 7300
-F 0 "CON1" H 5600 7550 60  0000 C CNN
+F 0 "9VAC1" H 5600 7550 60  0000 C CNN
 F 1 "BARREL_JACK" H 5600 7100 60  0000 C CNN
 F 2 "Connect:BARREL_JACK" H 5600 7300 60  0001 C CNN
@@
 NoConn ~ 5300 7300
 $Comp
-L JACK_STEREO J1
+L JACK_STEREO CT1
 U 1 1 547BF8A7
 P 1600 5150
-F 0 "J1" H 1225 5150 50  0000 R CNN
+F 0 "CT1" H 1225 5150 50  0000 R CNN
 F 1 "JACK_STEREO" H 1600 5400 50  0000 C CNN
 F 2 "diy_connectors:JACK_2.1_DC" H 1600 5150 60  0001 C CNN
@@
 	2100 5100 1950 5100
 $Comp
-L GND #PWR033
+L GND #PWR12
 U 1 1 547D4090
 P 3650 2100
-F 0 "#PWR033" H 3650 2100 30  0001 C CNN
+F 0 "#PWR12" H 3650 2100 30  0001 C CNN
 F 1 "GND" H 3650 2030 30  0001 C CNN
 F 2 "" H 3650 2100 60  0000 C CNN
@@
 $EndComp
 $Comp
-L GND #PWR034
+L GND #PWR13
 U 1 1 547D463A
 P 3650 3750
-F 0 "#PWR034" H 3650 3750 30  0001 C CNN
+F 0 "#PWR13" H 3650 3750 30  0001 C CNN
 F 1 "GND" H 3650 3680 30  0001 C CNN
 F 2 "" H 3650 3750 60  0000 C CNN
@@
 Wire Wire Line
 	3650 2000 3650 2100
+$Comp
+L GND #PWR30
+U 1 1 54909844
+P 9100 3550
+F 0 "#PWR30" H 9100 3300 60  0001 C CNN
+F 1 "GND" H 9100 3400 60  0000 C CNN
+F 2 "" H 9100 3550 60  0000 C CNN
+F 3 "" H 9100 3550 60  0000 C CNN
+	1    9100 3550
+	1    0    0    -1
+$EndComp
+Wire Wire Line
+	9350 3550 9350 3450
+Wire Wire Line
+	8850 3550 9350 3550
+Wire Wire Line
+	8850 3450 8850 3550
+Connection ~ 9100 3550
+Wire Wire Line
+	9000 3450 9000 3550
+Connection ~ 9000 3550
+Wire Wire Line
+	9200 3450 9200 3550
+Connection ~ 9200 3550
 $EndSCHEMATC

Commit message: Update kicad files
Other:
- note added: "22/12/2014"
- note added: "Shield schematic"
Changed lines of the file:
@@
 LIBS:valves
 LIBS:arduino_shieldsNCL
-LIBS:rfm12
-LIBS:diy_connectors
 LIBS:netbomo-cache
 EELAYER 25 0
@@
 	9200 3450 9200 3550
 Connection ~ 9200 3550
+Text Notes 8150 7650 0    60   ~ 0
+22/12/2014
+Text Notes 7400 7500 0    60   ~ 0
+Shield schematic
 $EndSCHEMATC
